File: hardware/_autosave-hardware.kicad_pcb (KiCad board)
At the start: 4 copper layers, 68.6 x 62.2 mm, 34 parts, among them J1 5034800800, U1 AP3429A, U2 ESP32-DEVKITC, U3 MPU-6050, U4 FDC2212

Commit message: PCB 10/25
Parts:
- renumbered H8 to GND
Changed lines of the file:
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@@
   (general
     (thickness 1.6)
-    (drawings 4)
+    (drawings 6)
     (tracks 285)
     (zones 0)
@@
     (tags "mounting hole 2.2mm m2 iso14580")
     (attr virtual)
-    (fp_text reference H8 (at 0 3.81) (layer F.SilkS)
+    (fp_text reference GND (at 0 3.81) (layer F.SilkS)
       (effects (font (size 1.5 1.5) (thickness 0.25)))
     )
@@
     )
   )
+  (dimension 62.23 (width 0.15) (layer Dwgs.User)
+    (gr_text "62.230 mm" (at 101.316001 126.365 270) (layer Dwgs.User)
+      (effects (font (size 1 1) (thickness 0.15)))
+    )
+    (feature1 (pts (xy 110.49 157.48) (xy 102.02958 157.48)))
+    (feature2 (pts (xy 110.49 95.25) (xy 102.02958 95.25)))
+    (crossbar (pts (xy 102.616001 95.25) (xy 102.616001 157.48)))
+    (arrow1a (pts (xy 102.616001 157.48) (xy 102.02958 156.353496)))
+    (arrow1b (pts (xy 102.616001 157.48) (xy 103.202422 156.353496)))
+    (arrow2a (pts (xy 102.616001 95.25) (xy 102.02958 96.376504)))
+    (arrow2b (pts (xy 102.616001 95.25) (xy 103.202422 96.376504)))
+  )
+  (dimension 68.58 (width 0.15) (layer Dwgs.User)
+    (gr_text "68.580 mm" (at 144.78 164.875999) (layer Dwgs.User)
+      (effects (font (size 1 1) (thickness 0.15)))
+    )
+    (feature1 (pts (xy 179.07 157.48) (xy 179.07 164.16242)))
+    (feature2 (pts (xy 110.49 157.48) (xy 110.49 164.16242)))
+    (crossbar (pts (xy 110.49 163.575999) (xy 179.07 163.575999)))
+    (arrow1a (pts (xy 179.07 163.575999) (xy 177.943496 164.16242)))
+    (arrow1b (pts (xy 179.07 163.575999) (xy 177.943496 162.989578)))
+    (arrow2a (pts (xy 110.49 163.575999) (xy 111.616504 164.16242)))
+    (arrow2b (pts (xy 110.49 163.575999) (xy 111.616504 162.989578)))
+  )
   (gr_line (start 179.07 95.25) (end 179.07 157.48) (layer Edge.Cuts) (width 0.1))
