File: hardware/hardware.kicad_pcb (KiCad board)
At the start: 4 copper layers, 68.6 x 62.2 mm, 34 parts, among them J1 5034800800, U1 AP3429A, U2 ESP32-DEVKITC, U3 MPU-6050, U4 FDC2212

Commit message: IO Output
Parts:
- added IO12: Solder, MountingHole:MountingHole_2.2mm_M2_ISO14580_Pad, F.Cu at (116.3, 128.0)
- added IO14: Solder, MountingHole:MountingHole_2.2mm_M2_ISO14580_Pad, F.Cu at (116.3, 134.6)
- moved R1 8.94 mm to (115.8, 142.9)
- moved J1 6.73 mm to (162.6, 153.4)
- moved D1 5.86 mm to (122.4, 142.1)
- moved GND1 4.07 mm to (116.3, 117.9)
- moved 5V1 2.80 mm to (116.3, 110.2)
- renumbered H5 to 3V3, H7 to 5V1, H9 to Cap1, H6 to Force1, H8 to GND1
Routing:
- net Net-(IO12-Pad1): track 0.00 -> 47.8 mm
- net Net-(IO14-Pad1): track 0.00 -> 42.5 mm
- net /~ACOU_RST: track 15.3 -> 22.0 mm
- net /MAIN_SDA: track 93.7 -> 100.4 mm
- net /ACOU_INT: track 19.9 -> 26.6 mm
- net /ACOU_PROG: track 19.9 -> 26.6 mm
- net /MAIN_SCL: track 92.2 -> 98.3 mm
- net Net-(D1-Pad2): track 4.08 -> 7.87 mm
- net +1V8: track 17.0 -> 13.8 mm
- net Net-(5V1-Pad1): track 69.3 -> 70.4 mm
- net /LED: track 32.7 -> 33.6 mm
- net GND: track 63.9 -> 64.7 mm
